File: dongle_board/dongle_board.sch (KiCad schematic (older format))
At the start: 5 parts

Commit message: Updated board schematic.
Parts:
- added U?: PCM2900CDBR, DB28, symbol dongle_board:PCM2900CDBR
- added Y?: Crystal, symbol Device:Crystal
Connections:
- new net: U?.20 (XTO), Y?.1
- new net: U?.21 (XTI), Y?.2
Changed lines of the file:
@@
 	1    0    0    -1
 $EndComp
+$Comp
+L dongle_board:PCM2900CDBR U?
+U 1 1 5D53B2A1
+P 6450 4600
+F 0 "U?" H 7750 4987 60  0000 C CNN
+F 1 "PCM2900CDBR" H 7750 4881 60  0000 C CNN
+F 2 "DB28" H 7750 4840 60  0001 C CNN
+F 3 "" H 6450 4600 60  0000 C CNN
+	1    6450 4600
+	1    0    0    -1
+$EndComp
+$Comp
+L Device:Crystal Y?
+U 1 1 5D54CB91
+P 9600 5350
+F 0 "Y?" V 9646 5219 50  0000 R CNN
+F 1 "Crystal" V 9555 5219 50  0000 R CNN
+F 2 "" H 9600 5350 50  0001 C CNN
+F 3 "~" H 9600 5350 50  0001 C CNN
+	1    9600 5350
+	0    -1   -1   0
+$EndComp
+Wire Wire Line
+	9050 5400 9400 5400
+Wire Wire Line
+	9400 5400 9400 5500
+Wire Wire Line
+	9400 5500 9600 5500
+Wire Wire Line
+	9050 5300 9400 5300
+Wire Wire Line
+	9400 5300 9400 5200
+Wire Wire Line
+	9400 5200 9600 5200
 $EndSCHEMATC
